File: hardware/stick/rev1-pcb/kicad/mcu.kicad_sch (KiCad schematic)
At the start: 11 parts, among them U4 nRF52840-QIAA-R7, Y1 32MHz, Y2 32.768kHz

Commit message: Add wired schematics, 3D cases, and solar relay KiCad project
Credstick Rev1 updates:
- Library tables (sym-lib-table, fp-lib-table) for custom libs
- Footprints: supercap cylindrical 14mm, piezo cantilever 25x5mm,
  3x3mm tactile switch
- Wired schematics with net labels and wire connections across all
  three sub-sheets (Power, MCU, Peripherals)
- Power sheet: VBUS→ESD→charge limiter→supercap→LDO chain with
  CC pull-downs, piezo rectifier, charge LED, and ILIM resistor
- MCU sheet: all GPIO assignments, crystal connections, DEC caps
- Peripherals: I2C pull-ups, SPI→FPC wiring, NFC matching network,
  button connections
- Supercap footprints now reference custom cylindrical footprint
- OpenSCAD parametric case (3d/credstick-case.scad): two-piece
  snap-fit, display window, button holes, USB-C cutout, keyring,
  LED window, piezo ventilation slot

Solar Relay (new KiCad project):
- Project with 4-sheet hierarchy: Power, MCU, NFC_Reader, IO
- Custom symbols: PN7150 (HVQFN-40 NFC reader), BQ25504 (QFN-20
  solar MPPT charger)
- Custom footprints: HVQFN-40 5x5mm, QFN-20 3.5x3.5mm
- PCB layout: 70x45mm board, 4-layer stackup, 3-turn NFC reader
  antenna on B.Cu, inner-layer keep-outs, component placement for
  nRF52840 + PN7150 + BQ25504 + 4 buttons + 3 LEDs + USB-C
- References shared credstick footprint library
- OpenSCAD case (3d/relay-case.scad): two-piece screw-together,
  solar cell window, button holes, LED windows, NFC tap zone
  marker on bottom face, M2 screw bosses

https://claude.ai/code/session_01TM1rFxbipYtvAkh4Vt7My7
Parts:
- added C12, C13, C15: 100nF, Capacitor_SMD:C_0402_1005Metric, symbol Device:C
- renumbered C16 to C14
Other:
- note added: "DEC1-DEC6: 100nF caps, place within 10mm of respective pins per nRF52840 PS §50"
- note added: "GPIO Assignment Table:"
- note added: "P0.02 AIN0 = VSCAP voltage sense (via divider) P0.13 = SPI SCK"
- note added: "P0.14 = SPI MOSI P0.15 = SPI CS P0.16 = EPD D/C P0.17 = EPD RST"
- note added: "P0.18 = EPD BUSY P0.19 = BTN_L P0.20 = BTN_R P0.21 = LED"
- note added: "P0.26 = I2C SDA P0.27 = I2C SCL NFC1/NFC2 = antenna"
- note added: "nRF52840 MCU — CRYSTAL + DECOUPLING + GPIO"
- note removed: "32.768kHz crystal: ABS07 series, 6.8pF load caps, for RTC + BLE timing"
- note removed: "32MHz crystal: ABM8 series, 12pF load caps"
- note removed: "DEC1-DEC6: Place decoupling caps within 10mm of respective pins per Nordic datasheet"
- note removed: "Pin assignments: P0.26/P0.27=I2C, P0.13-P0.18=SPI+EPD, P0.19/P0.20=Buttons, P0.21=LED"
- note removed: "nRF52840 MCU + CRYSTAL + DECOUPLING"
