File: hardware/stick/rev1-pcb/kicad/mcu.kicad_sch (KiCad schematic)
At the start: 14 parts, among them U4 nRF52840-QIAA-R7, Y1 32MHz, Y2 32.768kHz

Commit message: Replace ATECC608B with nano-SIM in push-push connector, add concurrent init
Replace the soldered-down ATECC608B secure element with a user-replaceable
nano-SIM card in a low-profile push-push connector (Molex 78800-0001,
1.25mm height). The SIM provides the same tamper-resistant functions
(P-256 ECDSA, key storage, monotonic counters) via standard ISO 7816
interface, but is field-swappable for identity transfer or replacement.
This makes the prototype robust enough for production use.

Hardware changes:
- Peripherals schematic: ATECC608B U5 → J3 nano-SIM connector
- I2C (SDA/SCL) → ISO 7816 (SIM_IO, SIM_CLK, SIM_RST, SIM_DET)
- MCU GPIO reassignment: P0.26=SIM_IO, P0.27=SIM_CLK, P0.22=SIM_RST,
  P0.24=SIM_DET
- New KiCad symbol (NanoSIM_PushPush) and footprint (NanoSIM_Molex_78800)
- BOM updated: SIM connector + card replaces ATECC608B
- 3D case: added SIM card slot cutout in side wall

Firmware changes:
- New sim_card.rs: async ISO 7816 T=0 driver over UARTE, with ATR
  parsing, applet selection, INTERNAL AUTHENTICATE signing, GET DATA
  for certificates/keys, and monotonic counter operations
- main.rs: concurrent initialization using embassy_futures::join3 —
  storage init, SIM card init, and display setup run in parallel
- Switched from blocking I2C (twim) to async UARTE for SIM communication
- atecc608b.rs marked deprecated (retained for reference)

https://claude.ai/code/session_01TM1rFxbipYtvAkh4Vt7My7
Other:
- note added: "P0.22 = SIM_RST (active low) P0.24 = SIM_DET (card detect, active low)"
- note added: "P0.26 = SIM_IO (UARTE half-duplex) P0.27 = SIM_CLK (PWM 3.25MHz)"
- note removed: "P0.26 = I2C SDA P0.27 = I2C SCL NFC1/NFC2 = antenna"
Changed lines of the file:
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@@
   (title_block
     (title "Briolette Credstick — MCU")
-    (date "2026-03-13")
-    (rev "1.0")
+    (date "2026-03-14")
+    (rev "1.1")
     (comment 1 "nRF52840 QFN-48 with crystals, decoupling, and all GPIO assignments")
   )
@@
   (hierarchical_label "GND" (shape passive) (at 25.4 152.4 180)
     (effects (font (size 1.27 1.27)) (justify right)) (uuid "hl-mcu-0002"))
-  (hierarchical_label "SDA" (shape bidirectional) (at 200.66 76.2 0)
+  (hierarchical_label "SIM_IO" (shape bidirectional) (at 200.66 76.2 0)
     (effects (font (size 1.27 1.27)) (justify left)) (uuid "hl-mcu-0003"))
-  (hierarchical_label "SCL" (shape output) (at 200.66 78.74 0)
+  (hierarchical_label "SIM_CLK" (shape output) (at 200.66 78.74 0)
     (effects (font (size 1.27 1.27)) (justify left)) (uuid "hl-mcu-0004"))
+  (hierarchical_label "SIM_RST" (shape output) (at 200.66 81.28 0)
+    (effects (font (size 1.27 1.27)) (justify left)) (uuid "hl-mcu-0004b"))
+  (hierarchical_label "SIM_DET" (shape input) (at 200.66 83.82 0)
+    (effects (font (size 1.27 1.27)) (justify left)) (uuid "hl-mcu-0004c"))
   (hierarchical_label "SPI_SCK" (shape output) (at 200.66 88.9 0)
     (effects (font (size 1.27 1.27)) (justify left)) (uuid "hl-mcu-0005"))
@@
   (label "~{RESET}" (at 76.2 124.46 0)
     (effects (font (size 1.27 1.27)) (justify left)) (uuid "nl-mcu-rst-r5"))
-  ;; I2C
-  (label "SDA" (at 142.24 149.86 0)
-    (effects (font (size 1.27 1.27)) (justify left)) (uuid "nl-mcu-sda"))
-  (label "SCL" (at 142.24 147.32 0)
-    (effects (font (size 1.27 1.27)) (justify left)) (uuid "nl-mcu-scl"))
+  ;; SIM card interface (was I2C — now ISO 7816)
+  ;; P0.26 → SIM_IO (UARTE0 TX/RX, half-duplex)
+  ;; P0.27 → SIM_CLK (PWM output, 3.25 MHz)
+  ;; P0.22 → SIM_RST (GPIO output, active low)
+  ;; P0.24 → SIM_DET (GPIO input, card detect, active low)
+  (label "SIM_IO" (at 142.24 149.86 0)
+    (effects (font (size 1.27 1.27)) (justify left)) (uuid "nl-mcu-simio"))
+  (label "SIM_CLK" (at 142.24 147.32 0)
+    (effects (font (size 1.27 1.27)) (justify left)) (uuid "nl-mcu-simclk"))
+  (label "SIM_RST" (at 142.24 144.78 0)
+    (effects (font (size 1.27 1.27)) (justify left)) (uuid "nl-mcu-simrst"))
+  (label "SIM_DET" (at 142.24 142.24 0)
+    (effects (font (size 1.27 1.27)) (justify left)) (uuid "nl-mcu-simdet"))
   ;; SPI (E-Ink)
-  (label "SPI_SCK" (at 142.24 142.24 0)
+  (label "SPI_SCK" (at 142.24 137.16 0)
     (effects (font (size 1.27 1.27)) (justify left)) (uuid "nl-mcu-sck"))
-  (label "SPI_MOSI" (at 142.24 139.7 0)
+  (label "SPI_MOSI" (at 142.24 134.62 0)
     (effects (font (size 1.27 1.27)) (justify left)) (uuid "nl-mcu-mosi"))
-  (label "SPI_CS" (at 142.24 137.16 0)
+  (label "SPI_CS" (at 142.24 132.08 0)
     (effects (font (size 1.27 1.27)) (justify left)) (uuid "nl-mcu-cs"))
-  (label "EPD_DC" (at 142.24 134.62 0)
+  (label "EPD_DC" (at 142.24 129.54 0)
     (effects (font (size 1.27 1.27)) (justify left)) (uuid "nl-mcu-dc"))
-  (label "EPD_RST" (at 142.24 132.08 0)
+  (label "EPD_RST" (at 142.24 127 0)
     (effects (font (size 1.27 1.27)) (justify left)) (uuid "nl-mcu-rst-epd"))
-  (label "EPD_BUSY" (at 142.24 129.54 0)
+  (label "EPD_BUSY" (at 142.24 124.46 0)
     (effects (font (size 1.27 1.27)) (justify left)) (uuid "nl-mcu-busy"))
   ;; Buttons + LED
-  (label "BTN_L" (at 142.24 124.46 0)
+  (label "BTN_L" (at 142.24 119.38 0)
     (effects (font (size 1.27 1.27)) (justify left)) (uuid "nl-mcu-btnl"))
-  (label "BTN_R" (at 142.24 121.92 0)
+  (label "BTN_R" (at 142.24 116.84 0)
     (effects (font (size 1.27 1.27)) (justify left)) (uuid "nl-mcu-btnr"))
-  (label "LED" (at 142.24 116.84 0)
+  (label "LED" (at 142.24 111.76 0)
     (effects (font (size 1.27 1.27)) (justify left)) (uuid "nl-mcu-led"))
   ;; ADC: supercap voltage sense (voltage divider on parent sheet)
-  (label "VSCAP_SENSE" (at 142.24 111.76 0)
+  (label "VSCAP_SENSE" (at 142.24 106.68 0)
     (effects (font (size 1.27 1.27)) (justify left)) (uuid "nl-mcu-ain0"))
   ;; DEC pins
@@
   ;; Output sheet labels
   (wire (pts (xy 142.24 149.86) (xy 200.66 76.2))
-    (stroke (width 0) (type default)) (uuid "w-mcu-sda-hl"))
+    (stroke (width 0) (type default)) (uuid "w-mcu-simio-hl"))
   (wire (pts (xy 142.24 147.32) (xy 200.66 78.74))
-    (stroke (width 0) (type default)) (uuid "w-mcu-scl-hl"))
+    (stroke (width 0) (type default)) (uuid "w-mcu-simclk-hl"))
   ;; ============================================================
   ;; Annotations
@@
     (uuid "txt-mcu-0008")
   )
-  (text "P0.26 = I2C SDA   P0.27 = I2C SCL   NFC1/NFC2 = antenna"
+  (text "P0.26 = SIM_IO (UARTE half-duplex)   P0.27 = SIM_CLK (PWM 3.25MHz)"
     (exclude_from_sim no)
     (at 25.4 40.64 0)
@@
     (uuid "txt-mcu-0009")
   )
+  (text "P0.22 = SIM_RST (active low)   P0.24 = SIM_DET (card detect, active low)"
+    (exclude_from_sim no)
+    (at 25.4 43.18 0)
+    (effects (font (size 1.27 1.27)))
+    (uuid "txt-mcu-0009b")
+  )
   (text "DEC1-DEC6: 100nF caps, place within 10mm of respective pins per nRF52840 PS §50"
     (exclude_from_sim no)
-    (at 25.4 43.18 0)
+    (at 25.4 45.72 0)
     (effects (font (size 1.27 1.27)))
     (uuid "txt-mcu-0010")
