File: hardware/stick/rev1-pcb/kicad/peripherals.kicad_sch (KiCad schematic)
At the start: 10 parts, among them J2 GDEY0154D67, SW1 BTN_LEFT, SW2 BTN_RIGHT, U5 ATECC608B-MAHDA-S

Commit message: Add wired schematics, 3D cases, and solar relay KiCad project
Credstick Rev1 updates:
- Library tables (sym-lib-table, fp-lib-table) for custom libs
- Footprints: supercap cylindrical 14mm, piezo cantilever 25x5mm,
  3x3mm tactile switch
- Wired schematics with net labels and wire connections across all
  three sub-sheets (Power, MCU, Peripherals)
- Power sheet: VBUS→ESD→charge limiter→supercap→LDO chain with
  CC pull-downs, piezo rectifier, charge LED, and ILIM resistor
- MCU sheet: all GPIO assignments, crystal connections, DEC caps
- Peripherals: I2C pull-ups, SPI→FPC wiring, NFC matching network,
  button connections
- Supercap footprints now reference custom cylindrical footprint
- OpenSCAD parametric case (3d/credstick-case.scad): two-piece
  snap-fit, display window, button holes, USB-C cutout, keyring,
  LED window, piezo ventilation slot

Solar Relay (new KiCad project):
- Project with 4-sheet hierarchy: Power, MCU, NFC_Reader, IO
- Custom symbols: PN7150 (HVQFN-40 NFC reader), BQ25504 (QFN-20
  solar MPPT charger)
- Custom footprints: HVQFN-40 5x5mm, QFN-20 3.5x3.5mm
- PCB layout: 70x45mm board, 4-layer stackup, 3-turn NFC reader
  antenna on B.Cu, inner-layer keep-outs, component placement for
  nRF52840 + PN7150 + BQ25504 + 4 buttons + 3 LEDs + USB-C
- References shared credstick footprint library
- OpenSCAD case (3d/relay-case.scad): two-piece screw-together,
  solar cell window, button holes, LED windows, NFC tap zone
  marker on bottom face, M2 screw bosses

https://claude.ai/code/session_01TM1rFxbipYtvAkh4Vt7My7
Parts:
- SW1, SW2: footprint Button_Switch_SMD:SW_SPST_PTS810 -> stick-lib:SW_SPST_3x3mm
Other:
- note added: "Buttons use nRF52840 internal pull-up (GPIO config). Active low. SW press → logic 0."
- note added: "E-Ink SPI: CS, D/C, RST, BUSY, SCK, MOSI (write-only, no MISO needed)"
- note added: "I2C Bus: SDA/SCL with 4.7kΩ pull-ups to VCC. ATECC608B default addr 0x60."
- note added: "NFC Antenna: Bottom copper layer PCB trace, 25×20mm rectangular spiral, 4-5 turns"
- note added: "NFC Matching: L1 (390nH) series with NFC1, C18/C19 (180pF) shunt to GND"
- note added: "Tune C18/C19 values for 13.56 MHz resonance. Start with 180pF, measure with VNA."
- note removed: "Buttons: Internal pull-up via nRF52840 GPIO config, active-low with hardware debounce"
- note removed: "E-Ink SPI: CS, D/C, RST, BUSY, SCK, MOSI (no MISO — write-only display)"
- note removed: "I2C Bus: SDA/SCL with 4.7kΩ pull-ups to VCC"
- note removed: "Matching network: L1 (390nH) in series, C18/C19 (180pF) shunt to GND — tune for 13.56 MHz"
- note removed: "NFC Antenna: PCB trace on B.Cu (bottom layer), 25x20mm rectangular spiral"
