File: hardware/stick/rev1-pcb/kicad/peripherals.kicad_sch (KiCad schematic)
At the start: 10 parts, among them J2 GDEY0154D67, SW1 BTN_LEFT, SW2 BTN_RIGHT, U5 ATECC608B-MAHDA-S

Commit message: Replace ATECC608B with nano-SIM in push-push connector, add concurrent init
Replace the soldered-down ATECC608B secure element with a user-replaceable
nano-SIM card in a low-profile push-push connector (Molex 78800-0001,
1.25mm height). The SIM provides the same tamper-resistant functions
(P-256 ECDSA, key storage, monotonic counters) via standard ISO 7816
interface, but is field-swappable for identity transfer or replacement.
This makes the prototype robust enough for production use.

Hardware changes:
- Peripherals schematic: ATECC608B U5 → J3 nano-SIM connector
- I2C (SDA/SCL) → ISO 7816 (SIM_IO, SIM_CLK, SIM_RST, SIM_DET)
- MCU GPIO reassignment: P0.26=SIM_IO, P0.27=SIM_CLK, P0.22=SIM_RST,
  P0.24=SIM_DET
- New KiCad symbol (NanoSIM_PushPush) and footprint (NanoSIM_Molex_78800)
- BOM updated: SIM connector + card replaces ATECC608B
- 3D case: added SIM card slot cutout in side wall

Firmware changes:
- New sim_card.rs: async ISO 7816 T=0 driver over UARTE, with ATR
  parsing, applet selection, INTERNAL AUTHENTICATE signing, GET DATA
  for certificates/keys, and monotonic counter operations
- main.rs: concurrent initialization using embassy_futures::join3 —
  storage init, SIM card init, and display setup run in parallel
- Switched from blocking I2C (twim) to async UARTE for SIM communication
- atecc608b.rs marked deprecated (retained for reference)

https://claude.ai/code/session_01TM1rFxbipYtvAkh4Vt7My7
Parts:
- J3: renamed from U5; value ATECC608B-MAHDA-S -> Nano-SIM Push-Push; footprint stick-lib:UDFN-8-2x3mm -> stick-lib:NanoSIM_Molex_78800; symbol stick-lib:ATECC608B -> stick-lib:NanoSIM_PushPush
- R6, R7: value 4.7k -> 10k
Other:
- note added: "ISO 7816 interface: SIM_IO (half-duplex data, 10k pull-up), SIM_CLK (3.25MHz PWM),"
- note added: "PERIPHERALS — SIM Card (ISO 7816), Display, Buttons, NFC Antenna"
- note added: "SIM Card: Nano-SIM (4FF) in low-profile push-push connector (Molex 78800-0001)."
- note added: "SIM_RST (active-low reset). VPP tied to VCC. Card detect (CD) with 10k pull-up."
- note removed: "I2C Bus: SDA/SCL with 4.7kΩ pull-ups to VCC. ATECC608B default addr 0x60."
- note removed: "PERIPHERALS — Secure Element, Display, Buttons, NFC Antenna"
- note removed: "Tune C18/C19 values for 13.56 MHz resonance. Start with 180pF, measure with VNA."
