File: hardware/stick/rev1-pcb/kicad/power.kicad_sch (KiCad schematic)
At the start: 15 parts, among them J1 USB4135-GF-A, U1 IP4292CZ12, U2 TPS2553, U3 AP2112K-3.3

Commit message: Add wired schematics, 3D cases, and solar relay KiCad project
Credstick Rev1 updates:
- Library tables (sym-lib-table, fp-lib-table) for custom libs
- Footprints: supercap cylindrical 14mm, piezo cantilever 25x5mm,
  3x3mm tactile switch
- Wired schematics with net labels and wire connections across all
  three sub-sheets (Power, MCU, Peripherals)
- Power sheet: VBUS→ESD→charge limiter→supercap→LDO chain with
  CC pull-downs, piezo rectifier, charge LED, and ILIM resistor
- MCU sheet: all GPIO assignments, crystal connections, DEC caps
- Peripherals: I2C pull-ups, SPI→FPC wiring, NFC matching network,
  button connections
- Supercap footprints now reference custom cylindrical footprint
- OpenSCAD parametric case (3d/credstick-case.scad): two-piece
  snap-fit, display window, button holes, USB-C cutout, keyring,
  LED window, piezo ventilation slot

Solar Relay (new KiCad project):
- Project with 4-sheet hierarchy: Power, MCU, NFC_Reader, IO
- Custom symbols: PN7150 (HVQFN-40 NFC reader), BQ25504 (QFN-20
  solar MPPT charger)
- Custom footprints: HVQFN-40 5x5mm, QFN-20 3.5x3.5mm
- PCB layout: 70x45mm board, 4-layer stackup, 3-turn NFC reader
  antenna on B.Cu, inner-layer keep-outs, component placement for
  nRF52840 + PN7150 + BQ25504 + 4 buttons + 3 LEDs + USB-C
- References shared credstick footprint library
- OpenSCAD case (3d/relay-case.scad): two-piece screw-together,
  solar cell window, button holes, LED windows, NFC tap zone
  marker on bottom face, M2 screw bosses

https://claude.ai/code/session_01TM1rFxbipYtvAkh4Vt7My7
Parts:
- added J3: PIEZO, stick-lib:Piezo_Cantilever_25x5mm, symbol Connector:Conn_01x02_Pin
- C1, C2: footprint (none) -> stick-lib:Supercap_Cylindrical_14mm
Other:
- note added: "Piezo harvester → BAT54S full-wave rectifier → 100µF buffer → VSCAP (trickle-charge)"
- note added: "R1 sets TPS2553 current limit: 10kΩ ≈ 1.05A, 47kΩ ≈ 0.21A"
- note added: "USB-C VBUS (5V) → IP4292CZ12 ESD → TPS2553 (1A limit) → Supercaps (2×5F 3V = 10F)"
- note added: "VSCAP (2.0-3.0V) → AP2112K-3.3 LDO → VCC (3.3V regulated)"
- note removed: "Piezo harvester (BAT54S rectifier + 100µF buffer) trickle-charges supercaps"
- note removed: "Supercap voltage (VSCAP, 2.0-3.0V) → AP2112K LDO → VCC (3.3V regulated)"
- note removed: "USB-C VBUS (5V) → ESD clamp → TPS2553 (1A limit) → Supercaps (2×5F 3V parallel = 10F)"
