File: hardware/relay/kicad/relay.kicad_pcb (KiCad board)
At the start: 4 copper layers, 70 x 45 mm, 22 parts, among them J1 USB4135-GF-A, SW1 KEY_1, SW10 KEY_9, SW11 KEY_DOT, SW12 KEY_0, SW13 KEY_OK, SW2 KEY_2, SW3 KEY_3, SW4 KEY_CLR, SW5 KEY_4, SW6 KEY_5, SW7 KEY_6, SW8 KEY_7, SW9 KEY_8, U1 nRF52840, U2 PN7150, U3 BQ25504, U4 AP2112K-3.3, U5 TCA8418

Commit message: Add missing passive footprints, fix firmware pin assignments
PCB changes (both boards):
- Add pad definitions to all footprints from library .kicad_mod files
- Add all missing passive components: decoupling caps, crystal load
  caps, LDO bypass caps, NFC matching network, pull-up/pull-down
  resistors, LED, piezo buffer cap, supercapacitor footprints
- Stick: 12 → 24 unique BOM parts on PCB
- Relay: 22 → 43 unique BOM parts on PCB

Firmware fixes:
- Stick: Realign display pins to match schematic (P0.15=CS, P0.16=DC,
  P0.17=RST, P0.18=BUSY), add TODO for SPIM peripheral init
- Relay: Add KEY_INT (P0.09) and KEY_RST (P0.10) pin definitions for
  TCA8418 keypad scanner, add TODO for I2C bus sharing

Docs:
- Update power-analysis.md: replace ATECC608B references with SIM card

Co-Authored-By: Claude Opus 4.6 (1M context) <noreply@anthropic.com>
Parts:
- added C1: 10F 3V, stick-lib:Supercap_Cylindrical_14mm, F.Cu at (25.0, -15.0)
- added C10: 100nF, Capacitor_SMD:C_0402_1005Metric, F.Cu at (-16.0, -3.50)
- added C11: 100nF, Capacitor_SMD:C_0402_1005Metric, F.Cu at (-16.0, 3.50)
- added C12: 100nF, Capacitor_SMD:C_0402_1005Metric, F.Cu at (-24.0, -3.50)
- added C13: 100nF, Capacitor_SMD:C_0402_1005Metric, F.Cu at (-24.0, 3.50)
- added C14: 100nF, Capacitor_SMD:C_0402_1005Metric, F.Cu at (-19.0, -4.50)
- added C15: 100nF, Capacitor_SMD:C_0402_1005Metric, F.Cu at (-21.0, -4.50)
- added C2: 10F 3V, stick-lib:Supercap_Cylindrical_14mm, F.Cu at (25.0, 15.0)
- added C20: 100nF, Capacitor_SMD:C_0402_1005Metric, F.Cu at (13.0, -2.00)
- added C21: 100nF, Capacitor_SMD:C_0402_1005Metric, F.Cu at (13.0, 0.00)
- added C22: 100nF, Capacitor_SMD:C_0402_1005Metric, F.Cu at (13.0, 2.00)
- added C23: 100nF, Capacitor_SMD:C_0402_1005Metric, F.Cu at (-16.0, -5.00)
- added C3: 10uF, Capacitor_SMD:C_0402_1005Metric, F.Cu at (-5.00, -8.00)
- added C30: 100nF, Capacitor_SMD:C_0402_1005Metric, F.Cu at (-5.00, -15.0)
- added C31: 4.7uF, Capacitor_SMD:C_0402_1005Metric, F.Cu at (-5.00, -13.0)
- added C32: 22uF, Capacitor_SMD:C_0805_2012Metric, F.Cu at (-11.0, -15.0)
- added C4: 10uF, Capacitor_SMD:C_0402_1005Metric, F.Cu at (-11.0, -8.00)
- added C40: 150pF, Capacitor_SMD:C_0402_1005Metric, F.Cu at (6.00, -3.00)
- added C41: 150pF, Capacitor_SMD:C_0402_1005Metric, F.Cu at (6.00, 3.00)
- added C42: 27pF, Capacitor_SMD:C_0402_1005Metric, F.Cu at (14.0, -3.00)
- added C43: 100nF, Capacitor_SMD:C_0402_1005Metric, F.Cu at (14.0, 3.00)
- added C44: 100nF, Capacitor_SMD:C_0402_1005Metric, F.Cu at (6.00, -5.00)
- added C5: 100uF, Capacitor_SMD:C_0805_2012Metric, F.Cu at (20.0, 18.0)
- added C6: 12pF, Capacitor_SMD:C_0402_1005Metric, F.Cu at (-15.0, 3.00)
- added C7: 12pF, Capacitor_SMD:C_0402_1005Metric, F.Cu at (-19.0, 3.00)
- added C8: 6.8pF, Capacitor_SMD:C_0402_1005Metric, F.Cu at (-15.0, 7.00)
- added C9: 6.8pF, Capacitor_SMD:C_0402_1005Metric, F.Cu at (-19.0, 7.00)
- added L1: 390nH, Inductor_SMD:L_0402_1005Metric, F.Cu at (6.00, 0.00)
- added L2: 2.2uH, Inductor_SMD:L_0402_1005Metric, F.Cu at (-8.00, -18.0)
- added R1: 10k, Resistor_SMD:R_0402_1005Metric, F.Cu at (3.00, 17.0)
- added R10: 5.76M, Resistor_SMD:R_0402_1005Metric, F.Cu at (-5.00, -17.0)
- added R11: 8.06M, Resistor_SMD:R_0402_1005Metric, F.Cu at (-5.00, -19.0)
- added R12: 5.76M, Resistor_SMD:R_0402_1005Metric, F.Cu at (-11.0, -17.0)
- added R13: 8.87M, Resistor_SMD:R_0402_1005Metric, F.Cu at (-11.0, -19.0)
- added R14: 5.76M, Resistor_SMD:R_0402_1005Metric, F.Cu at (-3.00, -15.0)
- added R15: 13.3M, Resistor_SMD:R_0402_1005Metric, F.Cu at (-3.00, -17.0)
- added R16: 5.76M, Resistor_SMD:R_0402_1005Metric, F.Cu at (-13.0, -15.0)
- added R17: 8.87M, Resistor_SMD:R_0402_1005Metric, F.Cu at (-13.0, -17.0)
- added R2: 1k, Resistor_SMD:R_0402_1005Metric, F.Cu at (-27.0, 10.0)
- added R20: 10R, Resistor_SMD:R_0402_1005Metric, F.Cu at (14.0, 0.00)
- added R3: 1k, Resistor_SMD:R_0402_1005Metric, F.Cu at (-23.0, 10.0)
- added R4: 1k, Resistor_SMD:R_0402_1005Metric, F.Cu at (-19.0, 10.0)
- added R5: 10k, Resistor_SMD:R_0402_1005Metric, F.Cu at (-23.0, -3.00)
- added R6: 5.1k, Resistor_SMD:R_0402_1005Metric, F.Cu at (-2.00, 17.0)
- added R7: 5.1k, Resistor_SMD:R_0402_1005Metric, F.Cu at (2.00, 17.0)
- added R8: 4.7k, Resistor_SMD:R_0402_1005Metric, F.Cu at (-17.0, -3.00)
- added R9: 4.7k, Resistor_SMD:R_0402_1005Metric, F.Cu at (-17.0, -5.00)

Commit message: Fix pre-fabrication review issues on both PCBs
Stick:
- Add piezo harvester footprint (J4, Piezo_Cantilever_25x5mm)
- Add NFC_ANT2 return trace on F.Cu from antenna exit via back to
  matching network area
- Fix 32MHz crystal footprint: 3215 (3.2x1.5mm) -> 3225 (3.2x2.5mm)
  to match ABM8 package

Relay:
- Add 5 missing components: BAT54S rectifier (D1), IP4292CZ12 ESD
  protection (U6), TPS2553 charge limiter (U7), solar cell pads (J2),
  piezo harvester (J3)
- Add both crystals: Y1 (32MHz, 3225 package) and Y2 (32.768kHz, 3215)
- Replace BQ25504 inductor L2 from 0402 to Coilcraft LPS4018 (4x4mm)
  matching the BQ25504 datasheet requirement
- Add missing 3rd 10uF bulk cap (C33)

Co-Authored-By: Claude Opus 4.6 (1M context) <noreply@anthropic.com>
Parts:
- added C33: 10uF, Capacitor_SMD:C_0402_1005Metric, F.Cu at (-8.00, -11.0)
- added D1: BAT54S, Package_TO_SOT_SMD:SOT-23, F.Cu at (20.0, 15.0)
- added J2: Solar_Cell, Connector_Wire:SolderWirePad_1x02_P5.08mm_D1.5mm, F.Cu at (-12.0, -20.0)
- added J3: PPA-1014, stick-lib:Piezo_Cantilever_25x5mm, F.Cu at (20.0, -20.0)
- added L2: 2.2uH, Inductor_SMD:L_Coilcraft_LPS4018, F.Cu at (-8.00, -18.0)
- added U6: IP4292CZ12, Package_SO:TSSOP-16_4.4x5mm_P0.65mm, F.Cu at (7.00, 20.0)
- added U7: TPS2553, Package_TO_SOT_SMD:SOT-23-6, F.Cu at (-7.00, 20.0)
- added Y1: 32MHz, Crystal:Crystal_SMD_3225-2Pin_3.2x2.5mm, F.Cu at (-17.0, 4.00)
- added Y2: 32.768kHz, Crystal:Crystal_SMD_3215-2Pin_3.2x1.5mm, F.Cu at (-17.0, 8.00)
Changed lines of the file:
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@@
     (pad "2" thru_hole circle (at 2.5 0) (size 2.0 2.0) (drill 1.0) (layers "*.Cu" "*.Mask"))
   )
+  (footprint "Package_TO_SOT_SMD:SOT-23"
+    (layer "F.Cu")
+    (at 20.0 15.0 0)
+    (property "Reference" "D1"
+      (at 0 -2.0 0)
+      (layer "F.SilkS")
+      (effects (font (size 0.6 0.6) (thickness 0.1)))
+    )
+    (property "Value" "BAT54S"
+      (at 0 2.5 0)
+      (layer "F.Fab")
+      (effects (font (size 0.6 0.6) (thickness 0.1)))
+    )
+    (pad "1" smd rect (at -0.95 1.1) (size 0.6 1.1) (layers "F.Cu" "F.Paste" "F.Mask"))
+    (pad "2" smd rect (at 0.95 1.1) (size 0.6 1.1) (layers "F.Cu" "F.Paste" "F.Mask"))
+    (pad "3" smd rect (at 0 -1.1) (size 0.6 1.1) (layers "F.Cu" "F.Paste" "F.Mask"))
+  )
+  (footprint "Package_SO:TSSOP-16_4.4x5mm_P0.65mm"
+    (layer "F.Cu")
+    (at 7.0 20.0 0)
+    (property "Reference" "U6"
+      (at 0 -4.5 0)
+      (layer "F.SilkS")
+      (effects (font (size 0.6 0.6) (thickness 0.1)))
+    )
+    (property "Value" "IP4292CZ12"
+      (at 0 4.5 0)
+      (layer "F.Fab")
+      (effects (font (size 0.6 0.6) (thickness 0.1)))
+    )
+    (pad "1" smd rect (at -2.275 2.95) (size 0.4 1.0) (layers "F.Cu" "F.Paste" "F.Mask"))
+    (pad "2" smd rect (at -1.625 2.95) (size 0.4 1.0) (layers "F.Cu" "F.Paste" "F.Mask"))
+    (pad "3" smd rect (at -0.975 2.95) (size 0.4 1.0) (layers "F.Cu" "F.Paste" "F.Mask"))
+    (pad "4" smd rect (at -0.325 2.95) (size 0.4 1.0) (layers "F.Cu" "F.Paste" "F.Mask"))
+    (pad "5" smd rect (at 0.325 2.95) (size 0.4 1.0) (layers "F.Cu" "F.Paste" "F.Mask"))
+    (pad "6" smd rect (at 0.975 2.95) (size 0.4 1.0) (layers "F.Cu" "F.Paste" "F.Mask"))
+    (pad "7" smd rect (at 1.625 2.95) (size 0.4 1.0) (layers "F.Cu" "F.Paste" "F.Mask"))
+    (pad "8" smd rect (at 2.275 2.95) (size 0.4 1.0) (layers "F.Cu" "F.Paste" "F.Mask"))
+    (pad "9" smd rect (at 2.275 -2.95) (size 0.4 1.0) (layers "F.Cu" "F.Paste" "F.Mask"))
+    (pad "10" smd rect (at 1.625 -2.95) (size 0.4 1.0) (layers "F.Cu" "F.Paste" "F.Mask"))
+    (pad "11" smd rect (at 0.975 -2.95) (size 0.4 1.0) (layers "F.Cu" "F.Paste" "F.Mask"))
+    (pad "12" smd rect (at 0.325 -2.95) (size 0.4 1.0) (layers "F.Cu" "F.Paste" "F.Mask"))
+    (pad "13" smd rect (at -0.325 -2.95) (size 0.4 1.0) (layers "F.Cu" "F.Paste" "F.Mask"))
+    (pad "14" smd rect (at -0.975 -2.95) (size 0.4 1.0) (layers "F.Cu" "F.Paste" "F.Mask"))
+    (pad "15" smd rect (at -1.625 -2.95) (size 0.4 1.0) (layers "F.Cu" "F.Paste" "F.Mask"))
+    (pad "16" smd rect (at -2.275 -2.95) (size 0.4 1.0) (layers "F.Cu" "F.Paste" "F.Mask"))
+  )
+  (footprint "Package_TO_SOT_SMD:SOT-23-6"
+    (layer "F.Cu")
+    (at -7.0 20.0 0)
+    (property "Reference" "U7"
+      (at 0 -3.0 0)
+      (layer "F.SilkS")
+      (effects (font (size 0.6 0.6) (thickness 0.1)))
+    )
+    (property "Value" "TPS2553"
+      (at 0 3.0 0)
+      (layer "F.Fab")
+      (effects (font (size 0.6 0.6) (thickness 0.1)))
+    )
+    (pad "1" smd rect (at -0.95 1.1) (size 0.6 1.1) (layers "F.Cu" "F.Paste" "F.Mask"))
+    (pad "2" smd rect (at 0 1.1) (size 0.6 1.1) (layers "F.Cu" "F.Paste" "F.Mask"))
+    (pad "3" smd rect (at 0.95 1.1) (size 0.6 1.1) (layers "F.Cu" "F.Paste" "F.Mask"))
+    (pad "4" smd rect (at 0.95 -1.1) (size 0.6 1.1) (layers "F.Cu" "F.Paste" "F.Mask"))
+    (pad "5" smd rect (at 0 -1.1) (size 0.6 1.1) (layers "F.Cu" "F.Paste" "F.Mask"))
+    (pad "6" smd rect (at -0.95 -1.1) (size 0.6 1.1) (layers "F.Cu" "F.Paste" "F.Mask"))
+  )
+  (footprint "Connector_Wire:SolderWirePad_1x02_P5.08mm_D1.5mm"
+    (layer "F.Cu")
+    (at -12.0 -20.0 0)
+    (property "Reference" "J2"
+      (at 0 -3.0 0)
+      (layer "F.SilkS")
+      (effects (font (size 0.6 0.6) (thickness 0.1)))
+    )
+    (property "Value" "Solar_Cell"
+      (at 0 3.0 0)
+      (layer "F.Fab")
+      (effects (font (size 0.6 0.6) (thickness 0.1)))
+    )
+    (pad "1" smd rect (at -2.54 0) (size 3.0 2.0) (layers "F.Cu" "F.Paste" "F.Mask"))
+    (pad "2" smd rect (at 2.54 0) (size 3.0 2.0) (layers "F.Cu" "F.Paste" "F.Mask"))
+  )
+  (footprint "stick-lib:Piezo_Cantilever_25x5mm"
+    (layer "F.Cu")
+    (at 20.0 -20.0 0)
+    (property "Reference" "J3"
+      (at 0 -5.0 0)
+      (layer "F.SilkS")
+      (effects (font (size 0.6 0.6) (thickness 0.1)))
+    )
+    (property "Value" "PPA-1014"
+      (at 0 5.0 0)
+      (layer "F.Fab")
+      (effects (font (size 0.6 0.6) (thickness 0.1)))
+    )
+    (pad "1" smd rect (at 11.0 -1.5) (size 2.0 1.5) (layers "F.Cu" "F.Paste" "F.Mask"))
+    (pad "2" smd rect (at 11.0 1.5) (size 2.0 1.5) (layers "F.Cu" "F.Paste" "F.Mask"))
+    (pad "MP" thru_hole circle (at 12.0 0) (size 1.6 1.6) (drill 1.0) (layers "*.Cu" "*.Mask"))
+  )
+  (footprint "Crystal:Crystal_SMD_3225-2Pin_3.2x2.5mm"
+    (layer "F.Cu")
+    (at -17.0 4.0 0)
+    (property "Reference" "Y1"
+      (at 0 -2.5 0)
+      (layer "F.SilkS")
+      (effects (font (size 0.6 0.6) (thickness 0.1)))
+    )
+    (property "Value" "32MHz"
+      (at 0 2.5 0)
+      (layer "F.Fab")
+      (effects (font (size 0.6 0.6) (thickness 0.1)))
+    )
+    (pad "1" smd rect (at -1.4 0) (size 1.8 1.4) (layers "F.Cu" "F.Paste" "F.Mask"))
+    (pad "2" smd rect (at 1.4 0) (size 1.8 1.4) (layers "F.Cu" "F.Paste" "F.Mask"))
+  )
+  (footprint "Crystal:Crystal_SMD_3215-2Pin_3.2x1.5mm"
+    (layer "F.Cu")
+    (at -17.0 8.0 0)
+    (property "Reference" "Y2"
+      (at 0 -2.0 0)
+      (layer "F.SilkS")
+      (effects (font (size 0.6 0.6) (thickness 0.1)))
+    )
+    (property "Value" "32.768kHz"
+      (at 0 2.0 0)
+      (layer "F.Fab")
+      (effects (font (size 0.6 0.6) (thickness 0.1)))
+    )
+    (pad "1" smd rect (at -1.3 0) (size 1.4 1.1) (layers "F.Cu" "F.Paste" "F.Mask"))
+    (pad "2" smd rect (at 1.3 0) (size 1.4 1.1) (layers "F.Cu" "F.Paste" "F.Mask"))
+  )
+  (footprint "Inductor_SMD:L_Coilcraft_LPS4018"
+    (layer "F.Cu")
+    (at -8.0 -18.0 0)
+    (property "Reference" "L2"
+      (at 0 -3.5 0)
+      (layer "F.SilkS")
+      (effects (font (size 0.6 0.6) (thickness 0.1)))
+    )
+    (property "Value" "2.2uH"
+      (at 0 3.5 0)
+      (layer "F.Fab")
+      (effects (font (size 0.6 0.6) (thickness 0.1)))
+    )
+    (pad "1" smd rect (at -1.5 0) (size 1.5 1.7) (layers "F.Cu" "F.Paste" "F.Mask"))
+    (pad "2" smd rect (at 1.5 0) (size 1.5 1.7) (layers "F.Cu" "F.Paste" "F.Mask"))
+  )
+  (footprint "Capacitor_SMD:C_0402_1005Metric"
+    (layer "F.Cu")
+    (at -8.0 -11.0 0)
+    (property "Reference" "C33"
+      (at 0 -1.2 0)
+      (layer "F.SilkS")
+      (effects (font (size 0.5 0.5) (thickness 0.08)))
+    )
+    (property "Value" "10uF"
+      (at 0 1.2 0)
+      (layer "F.Fab")
+      (effects (font (size 0.5 0.5) (thickness 0.08)))
+    )
+    (pad "1" smd roundrect (at -0.48 0) (size 0.56 0.62) (layers "F.Cu" "F.Paste" "F.Mask") (roundrect_rratio 0.25))
+    (pad "2" smd roundrect (at 0.48 0) (size 0.56 0.62) (layers "F.Cu" "F.Paste" "F.Mask") (roundrect_rratio 0.25))
+  )
 )
